Commit message: Fixed docker service calls & added mapping support to docker & added rviz packages

File: rob_ws/src/cario_static/urdf/cario.urdf.xacro (robot description, xacro)
@@ -42,5 +42,5 @@
   </xacro:if> -->
   <!-- Include the camera -->
-  <!-- <xacro:include filename="/home/antoine/rob1-tiago/src/pmb2_camera/src/camera/camera_macro.xacro" /> -->
+  <!-- <xacro:include filename="/home/antoine/rob1-tiago/src/cario_static/src/camera/camera_macro.xacro" /> -->
   <!-- Create the four cameras -->
   <!-- <xacro:camera name="camera_01" parent_link="base_link" pose_offset="0.2134410 0.0 0.6097676" orientation="0.0 ${pi/2} 0.0" />
@@ -48,5 +48,5 @@
   <xacro:camera name="camera_03" parent_link="base_link" pose_offset="0.0 0.2894102 0.6097676" orientation="-${pi/2} 0.0 0.0" />
   <xacro:camera name="camera_04" parent_link="base_link" pose_offset="0.0 -0.2894102 0.6097676" orientation="${pi/2} 0.0 0.0" /> -->
-  <xacro:include filename="$(find pmb2_camera)/src/urdf/plateform.xacro" />
+  <xacro:include filename="$(find cario_static)/urdf/plateform.xacro" />
   <xacro:plateform name="plateform" base_link="base_link" />
 </robot>

File: rob_ws/src/cario_static/urdf/plateform.xacro (robot description, xacro)
@@ -2,6 +2,6 @@
 <robot xmlns:xacro="http://ros.org/wiki/xacro">
     <xacro:macro name="plateform" params="name base_link">
-		<material name="blue">
-			<color rgba="0.2 0.2 1 1"/>
+		<material name="white">
+			<color rgba="0.9 0.9 0.9 1"/>
 		</material>
 		<!-- Plateform base visual annd collision mesh -->
@@ -15,7 +15,7 @@
 			<visual>
 				<geometry>
-					<mesh filename="$(find pmb2_camera)/src/urdf/robot_top_V1.stl"/>
+					<mesh filename="package://cario_static/urdf/robot_top_V1.stl"/>
 				</geometry>
-				<material name="blue"/>
+				<material name="white"/>
 			</visual>
 			<collision>
