Commit message: modify cario package dependencies & add pal_navigation_cfg_pmb2 to git

File: rob_ws/src/cario_robot/cario_description/robots/cario.urdf.xacro (robot description, xacro)
@@ -48,5 +48,5 @@
   <xacro:camera name="camera_03" parent_link="base_link" pose_offset="0.0 0.2894102 0.6097676" orientation="-${pi/2} 0.0 0.0" />
   <xacro:camera name="camera_04" parent_link="base_link" pose_offset="0.0 -0.2894102 0.6097676" orientation="${pi/2} 0.0 0.0" /> -->
-  <xacro:include filename="$(find cario_static)/urdf/plateform.xacro" />
+  <xacro:include filename="$(find cario_robot_model)/urdf/plateform.xacro" />
   <xacro:plateform name="plateform" base_link="base_link" />
 </robot>

File: rob_ws/src/cario_robot/cario_description/urdf/plateform/plateform.xacro (robot description, xacro)
@@ -15,5 +15,5 @@
 			<visual>
 				<geometry>
-					<mesh filename="package://cario_static/urdf/robot_top_V1.stl"/>
+					<mesh filename="package://cario_robot_model/urdf/robot_top_V1.stl"/>
 				</geometry>
 				<material name="white"/>

Commit message: modify cario packages

File: rob_ws/src/cario_robot/cario_description/robots/cario.urdf.xacro (robot description, xacro)
@@ -29,7 +29,7 @@
   <xacro:include filename="$(find pal_urdf_utils)/urdf/deg_to_rad.xacro" />
   <!-- Base -->
-  <xacro:include filename="$(find pmb2_description)/urdf/base/base_sensors.urdf.xacro" />
+  <xacro:include filename="$(find cario_description)/urdf/base/base_sensors.urdf.xacro" />
   <!-- Generic simulator_gazebo plugins -->
-  <xacro:include filename="$(find pmb2_description)/gazebo/gazebo.urdf.xacro" />
+  <xacro:include filename="$(find cario_description)/gazebo/gazebo.urdf.xacro" />
   <!-- Materials for visualization -->
   <xacro:include filename="$(find pal_urdf_utils)/urdf/materials.urdf.xacro" />
@@ -38,5 +38,5 @@
   <!-- RGBD Sensors -->
   <!-- <xacro:if value="${rgbd_sensors}">
-    <xacro:include filename="$(find pmb2_description)/urdf/cameras_add_on/cameras_add_on.urdf.xacro" />
+    <xacro:include filename="$(find cario_description)/urdf/cameras_add_on/cameras_add_on.urdf.xacro" />
     <xacro:cameras_add_on name="cameras_add_on" parent="base_link"/>
   </xacro:if> -->

File: rob_ws/src/cario_robot/cario_description/urdf/base/base.urdf.xacro (robot description, xacro)
@@ -13,9 +13,9 @@
 -->
 <robot xmlns:xacro="http://ros.org/wiki/xacro">
-  <xacro:include filename="$(find pmb2_description)/urdf/wheels/wheel.urdf.xacro"/>
-  <xacro:include filename="$(find pmb2_description)/urdf/wheels/caster.urdf.xacro"/>
-  <xacro:include filename="$(find pmb2_description)/urdf/sensors/imu.urdf.xacro"/>
-  <xacro:include filename="$(find pmb2_description)/urdf/objects/cover.urdf.xacro"/>
-  <xacro:include filename="$(find pmb2_description)/urdf/objects/antenna.urdf.xacro"/>
+  <xacro:include filename="$(find cario_description)/urdf/wheels/wheel.urdf.xacro"/>
+  <xacro:include filename="$(find cario_description)/urdf/wheels/caster.urdf.xacro"/>
+  <xacro:include filename="$(find cario_description)/urdf/sensors/imu.urdf.xacro"/>
+  <xacro:include filename="$(find cario_description)/urdf/objects/cover.urdf.xacro"/>
+  <xacro:include filename="$(find cario_description)/urdf/objects/antenna.urdf.xacro"/>
   <!-- Wheel characteristics -->
   <xacro:property name="wheel_radius"     value="0.0985"/>
@@ -45,5 +45,5 @@
         <origin xyz="0 0 0" rpy="0 0 0" />
         <geometry>
-          <mesh filename="package://pmb2_description/meshes/base/base.stl" />
+          <mesh filename="package://cario_description/meshes/base/base.stl" />
         </geometry>
         <material name="White" />
@@ -52,5 +52,5 @@
         <origin xyz="0 0 0" rpy="0 0 0" />
         <geometry>
-          <mesh filename="package://pmb2_description/meshes/base/base_collision.stl" />
+          <mesh filename="package://cario_description/meshes/base/base_collision.stl" />
         </geometry>
         <material name="White" />

File: rob_ws/src/cario_robot/cario_description/urdf/base/base_sensors.urdf.xacro (robot description, xacro)
@@ -13,13 +13,13 @@
 -->
 <robot xmlns:xacro="http://ros.org/wiki/xacro">
-  <xacro:include filename="$(find pmb2_description)/urdf/base/base.urdf.xacro"/>
-  <xacro:include filename="$(find pmb2_description)/urdf/sensors/hokuyo_urg_04lx_ug01_laser.urdf.xacro"/>
-  <xacro:include filename="$(find pmb2_description)/urdf/sensors/sick_tim551_laser.urdf.xacro"/>
-  <xacro:include filename="$(find pmb2_description)/urdf/sensors/sick_tim561_laser.urdf.xacro"/>
-  <xacro:include filename="$(find pmb2_description)/urdf/sensors/sick_tim571_laser.urdf.xacro"/>
-  <xacro:include filename="$(find pmb2_description)/urdf/sensors/ydlidar_tg30_laser.urdf.xacro"/>
-  <xacro:include filename="$(find pmb2_description)/urdf/sensors/ydlidar_tg15_laser.urdf.xacro"/>
-  <xacro:include filename="$(find pmb2_description)/urdf/sensors/range.urdf.xacro"/>
-  <xacro:include filename="$(find pmb2_description)/urdf/sensors/microphone.urdf.xacro"/>
+  <xacro:include filename="$(find cario_description)/urdf/base/base.urdf.xacro"/>
+  <xacro:include filename="$(find cario_description)/urdf/sensors/hokuyo_urg_04lx_ug01_laser.urdf.xacro"/>
+  <xacro:include filename="$(find cario_description)/urdf/sensors/sick_tim551_laser.urdf.xacro"/>
+  <xacro:include filename="$(find cario_description)/urdf/sensors/sick_tim561_laser.urdf.xacro"/>
+  <xacro:include filename="$(find cario_description)/urdf/sensors/sick_tim571_laser.urdf.xacro"/>
+  <!-- <xacro:include filename="$(find cario_description)/urdf/sensors/ydlidar_tg30_laser.urdf.xacro"/> -->
+  <!-- <xacro:include filename="$(find cario_description)/urdf/sensors/ydlidar_tg15_laser.urdf.xacro"/> -->
+  <xacro:include filename="$(find cario_description)/urdf/sensors/range.urdf.xacro"/>
+  <xacro:include filename="$(find cario_description)/urdf/sensors/microphone.urdf.xacro"/>
   <!-- Laser characteristics -->
   <xacro:property name="base_laser_x" value="0.202"/>
@@ -66,7 +66,5 @@
       </xacro:sick_tim571_laser>
     </xacro:if>
-    <xacro:if value="${laser_model == 'ydlidar-tg30'}">
-      <!-- Laser -->
-      <!-- Theoretic FOV = 360 -->
+    <!-- <xacro:if value="${laser_model == 'ydlidar-tg30'}">
       <xacro:ydlidar_tg30_laser name="${name}_laser" parent="${name}" ros_topic="scan_raw" update_rate="10" min_angle="${-65* deg_to_rad}" max_angle="${125 * deg_to_rad}" >
         <origin xyz="${base_laser_x} ${base_laser_y} ${base_laser_z}" rpy="0 0 ${ -30 * deg_to_rad }" />
@@ -74,10 +72,8 @@
     </xacro:if>
     <xacro:if value="${laser_model == 'ydlidar-tg15'}">
-      <!-- Laser -->
-      <!-- Theoretic FOV = 360 -->
       <xacro:ydlidar_tg15_laser name="${name}_laser" parent="${name}" ros_topic="scan_raw" update_rate="10" min_angle="${-65 * deg_to_rad}" max_angle="${125 * deg_to_rad}" >
         <origin xyz="${base_laser_x} ${base_laser_y} ${base_laser_z}" rpy="0 0 ${ -30 * deg_to_rad }" />
       </xacro:ydlidar_tg15_laser>
-    </xacro:if>
+    </xacro:if> -->
     <xacro:if value="${sonars}">
       <!-- Sonars -->

File: rob_ws/src/cario_robot/cario_description/urdf/cameras_add_on/cameras_add_on.urdf.xacro (robot description, xacro)
@@ -25,5 +25,5 @@
           <origin xyz="0 0 0" rpy="0 0 0"/>
           <geometry>
-            <mesh filename="package://pmb2_description/meshes/cameras_add_on/cameras_add_on.stl" scale="1 1 1"/>
+            <mesh filename="package://cario_description/meshes/cameras_add_on/cameras_add_on.stl" scale="1 1 1"/>
           </geometry>
           <material name="White" />
@@ -32,5 +32,5 @@
           <origin xyz="0 0 0" rpy="0 0 0" />
           <geometry>
-            <mesh filename="package://pmb2_description/meshes/cameras_add_on/cameras_add_on_collision.stl" scale="1 1 1"/>
+            <mesh filename="package://cario_description/meshes/cameras_add_on/cameras_add_on_collision.stl" scale="1 1 1"/>
           </geometry>
           <material name="White" />
@@ -44,4 +44,4 @@
       </joint>
     </xacro:macro>
-    <xacro:include filename="$(find pmb2_description)/urdf/sensors/courier.urdf.xacro" />
+    <xacro:include filename="$(find cario_description)/urdf/sensors/courier.urdf.xacro" />
   </robot>

File: rob_ws/src/cario_robot/cario_description/urdf/dock/dock.urdf.xacro (robot description, xacro)
@@ -13,5 +13,5 @@
 -->
 <robot xmlns:xacro="http://ros.org/wiki/xacro">
-  <xacro:include filename="$(find pmb2_description)/urdf/sensors/ir_emitter.urdf.xacro"/>
+  <xacro:include filename="$(find cario_description)/urdf/sensors/ir_emitter.urdf.xacro"/>
   <xacro:macro name="dock" params="name">
     <!-- Dock -->
@@ -25,6 +25,5 @@
         <origin xyz="0 0 0" rpy="0 0 0" />
         <geometry>
-          <mesh filename="package://pmb2_description/meshes/dock/dock.stl" />
-          <!--mesh filename="package://pmb2_description/meshes/dock/dock.dae" /-->
+          <mesh filename="package://cario_description/meshes/dock/dock.stl" />
         </geometry>
         <material name="LightGrey" />
@@ -33,5 +32,5 @@
         <origin xyz="0 0 0" rpy="0 0 0" />
         <geometry>
-          <mesh filename="package://pmb2_description/meshes/dock/dock_collision.stl" />
+          <mesh filename="package://cario_description/meshes/dock/dock_collision.stl" />
         </geometry>
         <material name="LightGrey" />

File: rob_ws/src/cario_robot/cario_description/urdf/objects/antenna.urdf.xacro (robot description, xacro)
@@ -25,5 +25,5 @@
         <origin xyz="0 0 0" rpy="0 0 0"/>
         <geometry>
-          <mesh filename="package://pmb2_description/meshes/objects/antenna.stl"/>
+          <mesh filename="package://cario_description/meshes/objects/antenna.stl"/>
         </geometry>
         <material name="Black"/>

File: rob_ws/src/cario_robot/cario_description/urdf/objects/cover.urdf.xacro (robot description, xacro)
@@ -25,5 +25,5 @@
         <origin xyz="0 0 0" rpy="0 0 0"/>
         <geometry>
-          <mesh filename="package://pmb2_description/meshes/base/base_ring.stl"/>
+          <mesh filename="package://cario_description/meshes/base/base_ring.stl"/>
         </geometry>
         <material name="Orange"/>

File: rob_ws/src/cario_robot/cario_description/urdf/sensors/bumper.urdf.xacro (robot description, xacro)
@@ -13,5 +13,5 @@
 -->
 <robot xmlns:xacro="http://ros.org/wiki/xacro">
-  <xacro:include filename="$(find pmb2_description)/urdf/sensors/bumper.gazebo.xacro" />
+  <xacro:include filename="$(find cario_description)/urdf/sensors/bumper.gazebo.xacro" />
   <xacro:macro name="bumper" params="name parent ros_topic update_rate *origin">
     <link name="${name}_link">
@@ -26,5 +26,5 @@
         <origin xyz="0 0 0" rpy="0 0 0" />
         <geometry>
-          <mesh filename="package://pmb2_description/meshes/sensors/bumper.stl"/>
+          <mesh filename="package://cario_description/meshes/sensors/bumper.stl"/>
         </geometry>
         <material name="DarkGrey"/>
@@ -33,5 +33,5 @@
         <origin xyz="0 0 0" rpy="0 0 0" />
         <geometry>
-          <mesh filename="package://pmb2_description/meshes/sensors/bumper_collision.stl"/>
+          <mesh filename="package://cario_description/meshes/sensors/bumper_collision.stl"/>
         </geometry>
         <material name="DarkGrey"/>

File: rob_ws/src/cario_robot/cario_description/urdf/sensors/courier.urdf.xacro (robot description, xacro)
@@ -13,8 +13,8 @@
 -->
 <robot xmlns:xacro="http://ros.org/wiki/xacro">
-  <xacro:include filename="$(find pmb2_description)/urdf/sensors/structure_sensor.urdf.xacro"/>
-  <xacro:include filename="$(find pmb2_description)/urdf/sensors/elp_rgb.urdf.xacro"/>
-  <xacro:property name="default_calibration_path" value="$(find pmb2_description)"/>
-  <xacro:property name="calibration_path" value="$(optenv pmb2_description_calibration_path ${default_calibration_path})"/>
+  <xacro:include filename="$(find cario_description)/urdf/sensors/structure_sensor.urdf.xacro"/>
+  <xacro:include filename="$(find cario_description)/urdf/sensors/elp_rgb.urdf.xacro"/>
+  <xacro:property name="default_calibration_path" value="$(find cario_description)"/>
+  <xacro:property name="calibration_path" value="$(optenv cario_description_calibration_path ${default_calibration_path})"/>
   <!-- base/roof RGBD calibratable characteristics -->
   <!-- spec: rgbd_z, rgbd_R and rgbd_P -->

File: rob_ws/src/cario_robot/cario_description/urdf/sensors/elp_rgb.urdf.xacro (robot description, xacro)
@@ -13,5 +13,5 @@
 -->
 <robot xmlns:xacro="http://ros.org/wiki/xacro">
- <xacro:include filename="$(find pmb2_description)/urdf/sensors/elp_rgb.gazebo.xacro" />
+ <xacro:include filename="$(find cario_description)/urdf/sensors/elp_rgb.gazebo.xacro" />
   <!-- Macro -->
   <xacro:macro name="elp_rgb" params="name parent *origin *optical_origin">
@@ -34,5 +34,5 @@
         <origin xyz="0 0 0" rpy="0 90 0"/>
         <geometry>
-          <mesh filename="package://pmb2_description/meshes/sensors/elp_camera.stl" scale="0.001 0.001 0.001"/>
+          <mesh filename="package://cario_description/meshes/sensors/elp_camera.stl" scale="0.001 0.001 0.001"/>
         </geometry>
         <material name="Grey" />

File: rob_ws/src/cario_robot/cario_description/urdf/sensors/hokuyo_urg_04lx_ug01_laser.urdf.xacro (robot description, xacro)
@@ -13,5 +13,5 @@
 -->
 <robot xmlns:xacro="http://ros.org/wiki/xacro">
-  <xacro:include filename="$(find pmb2_description)/urdf/sensors/hokuyo_urg_04lx_ug01_laser.gazebo.xacro" />
+  <xacro:include filename="$(find cario_description)/urdf/sensors/hokuyo_urg_04lx_ug01_laser.gazebo.xacro" />
   <xacro:macro name="hokuyo_urg_04lx_ug01_laser" params="name parent *origin ros_topic update_rate min_angle max_angle">
     <link name="${name}_link" type="laser">
@@ -26,5 +26,5 @@
         <origin xyz="0 0 0" rpy="0 0 0" />
         <geometry>
-          <mesh filename="package://pmb2_description/meshes/sensors/hokuyo_urg_04lx_ug01.stl"/>
+          <mesh filename="package://cario_description/meshes/sensors/hokuyo_urg_04lx_ug01.stl"/>
         </geometry>
         <material name="DarkGrey"/>

File: rob_ws/src/cario_robot/cario_description/urdf/sensors/range.urdf.xacro (robot description, xacro)
@@ -13,5 +13,5 @@
 -->
 <robot xmlns:xacro="http://ros.org/wiki/xacro">
-  <xacro:include filename="$(find pmb2_description)/urdf/sensors/range.gazebo.xacro" />
+  <xacro:include filename="$(find cario_description)/urdf/sensors/range.gazebo.xacro" />
   <xacro:macro name="range_sensor" params="name parent *origin ros_topic update_rate maxRange minRange fov radiation">
     <link name="${name}_link">
@@ -26,5 +26,5 @@
         <origin xyz="0 0 0" rpy="0 0 0" />
         <geometry>
-          <mesh filename="package://pmb2_description/meshes/sensors/srf05.stl"/>
+          <mesh filename="package://cario_description/meshes/sensors/srf05.stl"/>
         </geometry>
         <material name="DarkGrey"/>

File: rob_ws/src/cario_robot/cario_description/urdf/sensors/sick_tim551_laser.urdf.xacro (robot description, xacro)
@@ -13,5 +13,5 @@
 -->
 <robot xmlns:xacro="http://ros.org/wiki/xacro">
-  <xacro:include filename="$(find pmb2_description)/urdf/sensors/sick_tim551_laser.gazebo.xacro" />
+  <xacro:include filename="$(find cario_description)/urdf/sensors/sick_tim551_laser.gazebo.xacro" />
   <xacro:macro name="sick_tim551_laser" params="name parent *origin ros_topic update_rate min_angle max_angle">
      <link name="${name}_link" type="laser">
@@ -26,5 +26,5 @@
         <origin xyz="0 0 0" rpy="0 0 0" />
         <geometry>
-          <mesh filename="package://pmb2_description/meshes/sensors/sick_tim551.stl"/>
+          <mesh filename="package://cario_description/meshes/sensors/sick_tim551.stl"/>
         </geometry>
         <material name="DarkGrey"/>

File: rob_ws/src/cario_robot/cario_description/urdf/sensors/sick_tim561_laser.urdf.xacro (robot description, xacro)
@@ -13,5 +13,5 @@
 -->
 <robot xmlns:xacro="http://ros.org/wiki/xacro">
-  <xacro:include filename="$(find pmb2_description)/urdf/sensors/sick_tim561_laser.gazebo.xacro" />
+  <xacro:include filename="$(find cario_description)/urdf/sensors/sick_tim561_laser.gazebo.xacro" />
   <xacro:macro name="sick_tim561_laser" params="name parent *origin ros_topic update_rate min_angle max_angle">
      <link name="${name}_link" type="laser">
@@ -26,5 +26,5 @@
         <origin xyz="0 0 0" rpy="0 0 0" />
         <geometry>
-          <mesh filename="package://pmb2_description/meshes/sensors/sick_tim551.stl"/>
+          <mesh filename="package://cario_description/meshes/sensors/sick_tim551.stl"/>
         </geometry>
         <material name="DarkGrey"/>

File: rob_ws/src/cario_robot/cario_description/urdf/sensors/sick_tim571_laser.urdf.xacro (robot description, xacro)
@@ -13,5 +13,5 @@
 -->
 <robot xmlns:xacro="http://ros.org/wiki/xacro">
-  <xacro:include filename="$(find pmb2_description)/urdf/sensors/sick_tim571_laser.gazebo.xacro" />
+  <xacro:include filename="$(find cario_description)/urdf/sensors/sick_tim571_laser.gazebo.xacro" />
   <xacro:macro name="sick_tim571_laser" params="name parent *origin ros_topic update_rate min_angle max_angle">
      <link name="${name}_link" type="laser">
@@ -26,5 +26,5 @@
         <origin xyz="0 0 0" rpy="0 0 0" />
         <geometry>
-          <mesh filename="package://pmb2_description/meshes/sensors/sick_tim551.stl"/>
+          <mesh filename="package://cario_description/meshes/sensors/sick_tim551.stl"/>
         </geometry>
         <material name="DarkGrey"/>

File: rob_ws/src/cario_robot/cario_description/urdf/sensors/structure_sensor.urdf.xacro (robot description, xacro)
@@ -13,5 +13,5 @@
 -->
 <robot xmlns:xacro="http://ros.org/wiki/xacro">
-  <xacro:include filename="$(find pmb2_description)/urdf/sensors/structure_sensor.gazebo.xacro" />
+  <xacro:include filename="$(find cario_description)/urdf/sensors/structure_sensor.gazebo.xacro" />
   <!-- Macro -->
   <xacro:macro name="structure_sensor" params="name parent *origin *optical_origin">
@@ -36,5 +36,5 @@
         <origin xyz="0 0 0" rpy="0 0 0"/>
         <geometry>
-          <mesh filename="package://pmb2_description/meshes/sensors/structure_sensor.stl" scale="0.001 0.001 0.001" />
+          <mesh filename="package://cario_description/meshes/sensors/structure_sensor.stl" scale="0.001 0.001 0.001" />
         </geometry>
         <material name="Grey">

File: rob_ws/src/cario_robot/cario_description/urdf/sensors/ydlidar_tg15_laser.urdf.xacro (robot description, xacro)
@@ -8,5 +8,5 @@
 -->
 <robot xmlns:xacro="http://ros.org/wiki/xacro">
-  <xacro:include filename="$(find pmb2_description)/urdf/sensors/ydlidar_tg15_laser.gazebo.xacro" />
+  <xacro:include filename="$(find cario_description)/urdf/sensors/ydlidar_tg15_laser.gazebo.xacro" />
   <xacro:macro name="ydlidar_tg15_laser" params="name parent *origin ros_topic update_rate min_angle max_angle">
      <link name="${name}_link" type="laser">
@@ -21,5 +21,5 @@
         <origin xyz="0 0 0" rpy="0 0 0" />
         <geometry>
-          <mesh filename="package://pmb2_description/meshes/sensors/ydlidar.dae"/>
+          <mesh filename="package://cario_description/meshes/sensors/ydlidar.dae"/>
         </geometry>
         <material name="DarkGrey"/>

File: rob_ws/src/cario_robot/cario_description/urdf/sensors/ydlidar_tg30_laser.urdf.xacro (robot description, xacro)
@@ -8,5 +8,5 @@
 -->
 <robot xmlns:xacro="http://ros.org/wiki/xacro">
-  <xacro:include filename="$(find pmb2_description)/urdf/sensors/ydlidar_tg30_laser.gazebo.xacro" />
+  <xacro:include filename="$(find cario_description)/urdf/sensors/ydlidar_tg30_laser.gazebo.xacro" />
   <xacro:macro name="ydlidar_tg30_laser" params="name parent *origin ros_topic update_rate min_angle max_angle">
      <link name="${name}_link" type="laser">
@@ -21,5 +21,5 @@
         <origin xyz="0 0 0" rpy="0 0 0" />
         <geometry>
-          <mesh filename="package://pmb2_description/meshes/sensors/ydlidar.dae"/>
+          <mesh filename="package://cario_description/meshes/sensors/ydlidar.dae"/>
         </geometry>
         <material name="DarkGrey"/>

File: rob_ws/src/cario_robot/cario_description/urdf/wheels/caster.urdf.xacro (robot description, xacro)
@@ -13,5 +13,5 @@
 -->
 <robot xmlns:xacro="http://ros.org/wiki/xacro">
-  <xacro:include filename="$(find pmb2_description)/urdf/wheels/caster.gazebo.xacro"/>
+  <xacro:include filename="$(find cario_description)/urdf/wheels/caster.gazebo.xacro"/>
   <xacro:macro name="caster" params="side radius width separation_x separation_y offset_x offset_y offset_z parent">
     <link name="caster_${side}_1_link">
@@ -26,5 +26,5 @@
         <origin xyz="0 0 0" rpy="0 0 0"/>
         <geometry>
-          <mesh filename="package://pmb2_description/meshes/wheels/caster_1.stl"/>
+          <mesh filename="package://cario_description/meshes/wheels/caster_1.stl"/>
         </geometry>
         <material name="Grey"/>
@@ -48,5 +48,5 @@
         <origin xyz="0 0 0" rpy="0 0 0"/>
         <geometry>
-          <mesh filename="package://pmb2_description/meshes/wheels/caster_2.stl"/>
+          <mesh filename="package://cario_description/meshes/wheels/caster_2.stl"/>
         </geometry>
         <material name="DarkGrey"/>

File: rob_ws/src/cario_robot/cario_description/urdf/wheels/wheel.urdf.xacro (robot description, xacro)
@@ -13,6 +13,6 @@
 -->
 <robot xmlns:xacro="http://ros.org/wiki/xacro">
-  <xacro:include filename="$(find pmb2_description)/urdf/wheels/wheel.transmission.xacro"/>
-  <xacro:include filename="$(find pmb2_description)/urdf/wheels/wheel.gazebo.xacro"/>
+  <xacro:include filename="$(find cario_description)/urdf/wheels/wheel.transmission.xacro"/>
+  <xacro:include filename="$(find cario_description)/urdf/wheels/wheel.gazebo.xacro"/>
   <xacro:macro name="wheel" params="side reflect radius width torque velocity separation parent">
     <link name="wheel_${side}_link">
@@ -27,5 +27,5 @@
         <origin xyz="0 0 0" rpy="${-90.0 * (1 - reflect) * deg_to_rad} 0 0"/>
         <geometry>
-          <mesh filename="package://pmb2_description/meshes/wheels/wheel.stl"/>
+          <mesh filename="package://cario_description/meshes/wheels/wheel.stl"/>
         </geometry>
         <material name="DarkGrey"/>
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